File: schematic/msp430_gameboy.kicad_sch (KiCad schematic)
At the start: 27 parts, among them J1 OLED_SPI, J2 LiPo_Charger, SW1 SW_BTN_A, SW2 SW_BTN_B, SW3 SW_BTN_C, SW4 SW_BTN_D, SW5 SW_BTN_E, SW6 SW_BTN_F, SW7 SW_BTN_G, SW8 SW_BTN_H, U1 MSP430G2553, U2 SN74HC165N, U3 LM386N-1

Commit message: hardware: sync to rev 5.0 design, restructure as hardware-only repo
Repo split: this repo becomes the hardware side of the handheld project; the
firmware + 26-lesson course move to the companion software repo
(aradanmn/msp430-handheld).

- schematic/  update rev 4.0 -> rev 5.0 (OLED CS/DC/RST + SRAM + Flash) plus
              timestamped snapshots, from the software repo's newer design
- breadboard/ refresh guide + SVG to the current layout
- scripts/    refresh gen_kicad7.py to the current generator
- bom-*       add bill of materials (flat, structured, order CSV) at repo root
- wiring/     add per-build-phase wiring guides (phase-1 .. phase-4)
- README      rewrite for rev 5.0 + new layout, link to the software repo
- remove obsolete PUSH_TO_GITHUB.md local-push instructions

notes/ and logs/ retained verbatim as design history.
Parts:
- removed C1, C2: 100nF, symbol C
- removed J1: OLED_SPI, symbol Conn_01x04
- removed J2: LiPo_Charger, symbol Conn_01x04
- removed LS1: SP-3605 8R, symbol Speaker
- removed R1: 1k, symbol R
- removed R2, R3, R4, R5, R6, R7, R8, R9: 10k, symbol R
- removed RV1, RV2: 10k, symbol POT
- removed SW1: SW_BTN_A, symbol SW_Push
- removed SW2: SW_BTN_B, symbol SW_Push
- removed SW3: SW_BTN_C, symbol SW_Push
- removed SW4: SW_BTN_D, symbol SW_Push
- removed SW5: SW_BTN_E, symbol SW_Push
- removed SW6: SW_BTN_F, symbol SW_Push
- removed SW7: SW_BTN_G, symbol SW_Push
- removed SW8: SW_BTN_H, symbol SW_Push
- removed U1: MSP430G2553, symbol MSP430G2553
- removed U2: SN74HC165N, symbol SN74HC165N
- removed U3: LM386N-1, symbol LM386N
- added BT1: LiPo_JST, symbol Connector:Conn_01x02_Pin
- added C1, C2, C3, C4: 100nF, symbol Device:C
- added C10, C11: 4.7uF 10V X5R, symbol Device:C
- added C12: 100nF 16V X7R, symbol Device:C
- added C13: 10uF 16V X5R, symbol Device:C
- added C14: 10uF 10V X5R, symbol Device:C
- added C15, C16, C9: 1uF 10V X5R, symbol Device:C
- added C5, C6: 10uF, symbol Device:C
- added C7: 220uF, symbol Device:C
- added C8: 100nF 10V X5R, symbol Device:C
- added D1: LED_RED 0603, symbol Device:LED
- added D2: LED_GRN 0603, symbol Device:LED
- added DS1: OLED-128O064D, symbol Display_Graphic:OLED-128O064D
- added J4: USB_B_Micro, symbol Connector:USB_B_Micro
- added LS1: SP-3605, symbol Device:Speaker
- added Q1, Q2: AO3400, symbol Transistor_FET:Q_NMOS_GSD
- added R1: 1k, symbol Device:R
- added R10: 910k 1% 0402, symbol Device:R
- added R11: 2k 1%, symbol Device:R
- added R12, R13: 1k 5%, symbol Device:R
- added R2, R3, R4, R5, R6, R7, R8, R9: 10k, symbol Device:R
- added SW1: BTN_A, symbol Switch:SW_Push
- added SW2: BTN_B, symbol Switch:SW_Push
- added SW3: BTN_C, symbol Switch:SW_Push
- added SW4: BTN_D, symbol Switch:SW_Push
- added SW5: BTN_E, symbol Switch:SW_Push
- added SW6: BTN_F, symbol Switch:SW_Push
- added SW7: BTN_G, symbol Switch:SW_Push
- added SW8: BTN_H, symbol Switch:SW_Push
- added U1: MSP430G2553, symbol MCU_Texas_MSP430:MSP430G2553IN20
- added U2: SN74HC165N, symbol 74xx:74HC165
- added U3: LM386N-1, symbol Amplifier_Audio:LM386
- added U4: 23LC1024-I/P, symbol SRAM_23LC1024
- added U5: W25Q128JVSSIQ, symbol Memory_Flash:W25Q128JVS
- added U7: TP4056-42-ESOP8, symbol Battery_Management:TP4056-42-ESOP8
- added U8: DW01A, symbol Battery_Management:DW01A
Connections:
- net GND: now also C1.2, C10.2, C11.1, C12.2, C13.2, C14.2, C2.2, C3.2, C4.2, DS1.1 (GND), DS1.10 (BS0), DS1.11 (BS1), DS1.29 (VLSS), DS1.30 (GND), DS1.8 (VSS), J4.5 (GND), J4.6 (Shield), LS1.2, Q2.2 (S), R11.2, SW1.1, SW2.1, SW3.1, SW4.1, SW5.1, SW6.1, SW7.1, SW8.1, U1.20 (DVSS), U2.10 (DS), U2.15 (~{CE}), U2.8 (GND), U3.2 (-), U3.4 (GND), U4.4 (GND), U5.4 (GND), U7.3 (GND), U7.9 (EPAD), U8.2 (CS), U8.6 (GND)
- net MISO: now also U1.14 (TDI/TCLK/UCB0SOMI/UCB0SCL/TA0.1/CA6/A6/P1.6), U2.9 (Q7), U4.2 (SO), U5.2 (DO/IO_{1})
- net MOSI: now also DS1.19 (D1), U1.15 (TDO/TDI/UCB0SIMO/UCB0SDA/CAOUT/CA7/A7/P1.7), U4.5 (SI), U5.5 (DI/IO_{0})
- net PWM_OUT: now also R1.1, U1.4 (UCA0TXD/UCA0SIMO/TA0.1/CA2/A2/P1.2)
- net SCK: now also DS1.18 (D0), U1.7 (TMS/UCB0CLK/UCA0STE/TA0.0/CA5/A5/P1.5), U2.2 (CP), U4.6 (SCK), U5.6 (CLK)
- net SH_LD: now also U1.13 (P2.5/TA1.2), U2.1 (~{PL})
- net VCC: now also C1.1, C2.1, C3.1, C4.1, C6.1, C8.1, C9.1, DS1.12 (BS2), R10.1, R12.1, R13.1, R2.1, R3.1, R4.1, R5.1, R6.1, R7.1, R8.1, R9.1, U1.1 (DVCC), U2.16 (VCC), U3.6 (V+), U4.7 (~{HOLD}), U4.8 (VCC), U5.3 (~{WP}/IO_{2}), U5.7 (~{HOLD}/~{RESET}/IO_{3}), U5.8 (VCC)
- new net: C8.2, DS1.9 (VDD)
- new net: R2.2, SW1.2, U2.11 (D0)
- new net: R11.1, U7.2 (PROG)
- new net: R5.2, SW4.2, U2.14 (D3)
- new net: C11.2, DS1.27 (VCOMH)
- new net: R6.2, SW5.2, U2.3 (D4)
- new net: R4.2, SW3.2, U2.13 (D2)
- new net: R8.2, SW7.2, U2.5 (D6)
- new net: D2.1 (K), U7.6 (~{STDBY})
- new net: D2.2 (A), R13.2
- new net: Q2.1 (G), U8.3 (OC)
- new net: Q1.3 (D), Q2.3 (D)
- new net: R3.2, SW2.2, U2.12 (D1)
- new net: C9.2, DS1.6 (VBAT)
- new net: C5.1, R1.2
- new net: C16.1, DS1.5 (C1N)
- new net: C16.2, DS1.4 (C1P)
- new net: D1.1 (K), U7.7 (~{CHRG})
- new net: D1.2 (A), R12.2
- new net: BT1.2 (Pin_2), Q1.2 (S)
- new net: C15.1, DS1.2 (C2N)
- new net: C15.2, DS1.3 (C2P)
- new net: R7.2, SW6.2, U2.4 (D5)
- new net: R9.2, SW8.2, U2.6 (D7)
- new net: C7.1, LS1.1
- new net: C7.2, U3.5
- new net: C10.1, DS1.28 (VCC)
- new net: DS1.26 (IREF), R10.2
- new net: C5.2, U3.3 (+)
- new net: C6.2, U3.7 (BYPASS)
- new net: Q1.1 (G), U8.1 (OD)
- new net FLASH_CS: U1.12 (P2.4/TA1.2), U5.1 (~{CS})
- new net OLED_CS: DS1.13 (~{CS}), U1.8 (P2.0/TA1.0)
- new net OLED_DC: DS1.15 (D/~{C}), U1.9 (P2.1/TA1.1)
- new net OLED_RST: DS1.14 (~{RES}), U1.10 (P2.2/TA1.1)
- new net SRAM_CS: U1.11 (P2.3/TA1.0), U4.1 (~{CS})
- new net VBAT: BT1.1 (Pin_1), C14.1, U7.5 (BAT), U8.5 (VCC)
- new net VBUS: C12.1, C13.1, J4.1 (VBUS), U7.1 (TEMP), U7.4 (V_{CC}), U7.8 (CE)
- no-connect marks 17 -> 24
Other:
- title: MSP430G2553 Game Boy -> MSP430G2553 Handheld Game Console
